Commit message: Motion of the robot is tested with the scripts and implemented in the regular twist commands with assisted_teleop.py

File: description/gazebo_control.xacro (robot description, xacro)
@@ -7,5 +7,5 @@
             <right_joint>right_wheel_joint</right_joint>
             <wheel_separation>0.25</wheel_separation>
-            <wheel_radius>0.055</wheel_radius>
+            <wheel_radius>0.061</wheel_radius>
             <!-- Limits -->
             <!-- <max_wheel_torque>200</max_wheel_torque> -->

File: description/robot_core.xacro (robot description, xacro)
@@ -6,5 +6,5 @@
     <xacro:property name="chassis_height" value="0.11"/>
     <xacro:property name="chassis_mass" value="2.0"/>
-    <xacro:property name="wheel_radius" value="0.055"/>
+    <xacro:property name="wheel_radius" value="0.061"/>
     <xacro:property name="wheel_thickness" value="0.040"/>
     <xacro:property name="wheel_mass" value="0.05"/>
